File: Version_0.3/3_Phase_Controller_V0.3.sch (EAGLE design)
At the start: 51 parts

Commit message: Testing ignore
Parts:
- added U$6: DRV8353RH, Brad_Library:DRV8353RH
Connections:
- removed net N$34: C3.2, U$3.CB
- new net N$10: C5.2, U$6.DVDD
- new net N$11: C8.1, U$6.VDRAIN
- new net N$12: C8.2, U$6.VCP
- new net N$13: C3.1, U$6.VGLS
- net CAL: no longer U$3.CAL
- net DVDD: now also U$6.VREF; no longer C5.1, U$3.DVDD, U$3.VREF
- net EN_GATE: now also U$6.ENABLE; no longer U$3.ENABLE
- net FAULT: now also U$6.N_FAULT; no longer U$3.N_FAULT
- net GH_A: now also U$6.GHA; no longer U$3.GHA
- net GH_B: now also U$6.GHB; no longer U$3.GHB
- net GH_C: now also U$6.GHC; no longer U$3.GHC
- net GL_A: now also U$6.GLA; no longer U$3.GLA
- net GL_B: now also U$6.GLB; no longer U$3.GLB
- net GL_C: now also U$6.GLC; no longer U$3.GLC
- net GND: now also C3.2, C5.1, U$6.AGND, U$6.DGND, U$6.GND, U$6.PGND, U$6.SNA, U$6.SNB; no longer C2.1, C5.2, U$3.AGND, U$3.BGND, U$3.DGND, U$3.SNA, U$3.SNB
- net INH_A: now also U$6.INHA; no longer U$3.INHA
- net INH_B: now also U$6.INHB; no longer U$3.INHB
- net INH_C: now also U$6.INHC; no longer U$3.INHC
- net INL_A: now also U$6.INLA; no longer U$3.INLA
- net INL_B: now also U$6.INLB; no longer U$3.INLB
- net INL_C: now also U$6.INLC; no longer U$3.INLC
- net N$2: now also U$6.GAIN; no longer U$3.GAIN
- net N$21: now also U$6.SW; no longer C3.1, U$3.SW
- net N$22: now also U$6.CPH; no longer U$3.CPH
- net N$23: now also U$6.CPL; no longer U$3.CPL
- net N$5: now also U$6.VDS; no longer U$3.VDS
- net N$6: now also R2.1; no longer C8.1, U$3.VCP
- net N$7: now also U$6.IDRIVE; no longer U$3.IDRIVE
- net N$8: now also U$6.MODE; no longer U$3.MODE
- net PHASA: now also U$6.SHA; no longer U$3.SHA
- net PHASB: now also U$6.SHB; no longer U$3.SHB
- net PHASC: now also U$6.SHC; no longer U$3.SHC
- net PVDD: now also U$6.VM; no longer C2.2, C8.2, U$3.VDRAIN, U$3.VM
- net SN1: now also U$6.SPA; no longer U$3.SPA
- net SN2: now also U$6.SPB; no longer U$3.SPB
- net SO1: now also U$6.SOC; no longer U$3.SOC
- net SO2: now also U$6.SOB; no longer U$3.SOB
- net VCC: no longer R2.1
Other:
- moved on the sheet: C1, C10, C12, C16, C2, C3, C5, C6, C8, C9, L1, R10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
