File: Version_0.3/3_Phase_Controller_V0.3.brd (EAGLE design)
At the start: 80 x 57.5 mm, 51 parts

Commit message: Testing ignore
Parts:
- added U$6: DRV8353RH, Brad_Library:VQFN-RGZ0048A
Connections:
- removed net N$34: C3.2, U$3.44
- new net N$10: C5.2, U$6.40
- new net N$11: C8.1, U$6.6
- new net N$12: C8.2, U$6.7
- new net N$13: C3.1, U$6.2
- net CAL: no longer U$3.34
- net DVDD: now also U$6.26; no longer C5.1, U$3.26, U$3.36
- net EN_GATE: now also U$6.33; no longer U$3.33
- net FAULT: now also U$6.28; no longer U$3.28
- net GH_A: now also U$6.8; no longer U$3.8
- net GH_B: now also U$6.17; no longer U$3.17
- net GH_C: now also U$6.18; no longer U$3.18
- net GL_A: now also U$6.10; no longer U$3.10
- net GL_B: now also U$6.15; no longer U$3.15
- net GL_C: now also U$6.20; no longer U$3.20
- net GND: now also C3.2, C5.1, U$6.1, U$6.12, U$6.13, U$6.27, U$6.41, U$6.GND_PAD; no longer C2.1, C5.2, U$3.12, U$3.13, U$3.27, U$3.35, U$3.43
- net INH_A: now also U$6.34; no longer U$3.37
- net INH_B: now also U$6.36; no longer U$3.39
- net INH_C: now also U$6.38; no longer U$3.41
- net INL_A: now also U$6.35; no longer U$3.38
- net INL_B: now also U$6.37; no longer U$3.40
- net INL_C: now also U$6.39; no longer U$3.42
- net N$2: now also U$6.32; no longer U$3.32
- net N$21: now also U$6.42; no longer C3.1, U$3.45
- net N$22: now also U$6.4; no longer U$3.4
- net N$23: now also U$6.3; no longer U$3.3
- net N$5: now also U$6.31; no longer U$3.31
- net N$6: now also R2.1; no longer C8.1, U$3.5
- net N$7: now also U$6.30; no longer U$3.30
- net N$8: now also U$6.29; no longer U$3.29
- net PHASA: now also U$6.9; no longer U$3.9
- net PHASB: now also U$6.16; no longer U$3.16
- net PHASC: now also U$6.19; no longer U$3.19
- net PVDD: now also U$6.5; no longer C2.2, C8.2, U$3.6, U$3.7
- net SN1: now also U$6.11; no longer U$3.11
- net SN2: now also U$6.14; no longer U$3.14
- net SO1: now also U$6.23; no longer U$3.23
- net SO2: now also U$6.24; no longer U$3.24
- net VCC: no longer R2.1
Routing:
- net PVDD: track 91.6 -> 36.5 mm
- net PHASC: track 28.4 -> 0.00 mm
- net PHASA: track 21.9 -> 0.00 mm
- net GND: track 73.3 -> 54.6 mm, vias 73 -> 70
- net PHASB: track 15.2 -> 0.00 mm
- net INH_A: track 31.8 -> 17.8 mm
- net N$21: track 17.6 -> 4.15 mm
- net SN1: track 16.2 -> 4.15 mm
- net DVDD: track 40.7 -> 31.1 mm
- net N$6: track 7.35 -> 0.00 mm
- net N$34: track 6.31 -> 0.00 mm
- net N$8: track 5.78 -> 0.35 mm
- net N$22: track 6.25 -> 1.40 mm
- net N$7: track 16.1 -> 11.2 mm
- net GL_B: track 13.5 -> 8.87 mm
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
Commit message: Version 0.3 finished and ordered.
Parts:
- removed U$6: DRV8353RH, Brad_Library:VQFN-RGZ0048A
- added C17: 10 u, rcl:C1206
- added C18: 1 u, rcl:C0805
- added R13: 10 k, rcl:R0603
- C10: value 1 u -> 0.1 u
- C11, C4: value 220 u -> 1 u; device Brad_Library:C050-045X075 -> rcl:C0805
- C13: value 10 u -> 220 u; device rcl:C1206 -> Brad_Library:C050-045X075
- C14: value 10 u -> 1 u; device rcl:C1206 -> rcl:C0805
- C16: value 1 u -> 10 u; device rcl:C0805 -> rcl:C1206
- C2: value Cin -> 0.47u
- C3: value 0.1 u -> Cin
- C5: value 1 u -> 0.01u
- C6: value 47 n -> 220 u; device rcl:C0805 -> Brad_Library:C050-045X075
- C7: value 220 u -> 0.1 u; device Brad_Library:C050-045X075 -> rcl:C0805
- C8: value 1 u -> 47 n
- C9: value 0.1 u -> 220 u; device rcl:C0805 -> Brad_Library:C050-045X075
- R12: value 10 k -> 0
- R2: value 31.6 k -> 43k
- R3: value 100 k -> 100k; device rcl:R0805 -> rcl:R0603
- R4: value 10 k -> 100 k; device rcl:R0603 -> rcl:R0805
- R5: value 0 -> 100 k; device rcl:R0603 -> rcl:R0805
- R8: value 47 k -> 0
- R9: value 0 -> 47 k
- U$3: value DRV8323RH -> DRV8353RH
- moved C13 30.7 mm to (-23.4, -4.92), turned to 90 degrees
- moved C11 28.5 mm to (5.04, -3.27), turned to 270 degrees
- moved C15 26.9 mm to (6.48, -11.9), turned to 270 degrees
- moved C14 17.6 mm to (-5.75, -8.47), turned to 90 degrees
- moved C16 17.3 mm to (11.5, -11.9)
- moved R5 16.7 mm to (-6.62, 7.25)
- moved C4 15.3 mm to (1.12, 8.97), turned to 270 degrees
- moved C10 13.5 mm to (-8.15, -0.59), turned to 180 degrees
- moved C7 10.4 mm to (-8.65, 3.48), turned to 180 degrees
- moved C5 10.4 mm to (-4.00, 6.38), turned to 0 degrees
- moved R12 9.06 mm to (16.0, -1.85)
- moved R3 8.15 mm to (-10.3, 7.53), turned to 90 degrees
- moved C9 7.79 mm to (-18.5, 0.08), turned to 90 degrees
- moved R8 7.67 mm to (14.4, 3.65)
- moved R2 6.90 mm to (-12.3, 9.90), turned to 0 degrees
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Connections:
- removed net N$10: C5.2, U$6.40
- removed net N$11: C8.1, U$6.6
- removed net N$35: R3.2, U$3.48
- new net N$14: R5.1, U$3.46
- new net N$15: R4.1, U$3.47
- new net N$9: C2.2, U$3.44
- net DVDD: now also C11.2, C4.2, R13.1, R8.2, U$3.26, U$3.40; no longer C10.2, R12.1, R5.2, U$6.26
- net EN_GATE: now also U$3.33; no longer U$6.33
- net FAULT: now also R13.2, U$3.28; no longer R12.2, U$6.28
- net GH_A: now also U$3.8; no longer U$6.8
- net GH_B: now also U$3.17; no longer U$6.17
- net GH_C: now also U$3.18; no longer U$6.18
- net GL_A: now also U$3.10; no longer U$6.10
- net GL_B: now also U$3.15; no longer U$6.15
- net GL_C: now also U$3.20; no longer U$6.20
- net GND: now also C10.2, C11.1, C13.2, C14.2, C17.1, C18.1, C2.1, C3.1, C4.1, C6.2, R12.1, R2.1, R5.2, U$3.1, U$3.12, U$3.13, U$3.27, U$3.41; no longer C10.1, C11.2, C12.2, C13.1, C14.1, C3.2, C4.2, C5.1, R4.2, R8.1, U$3.2, U$6.1, U$6.12, U$6.13, U$6.27, U$6.41, U$6.GND_PAD
- net INH_A: now also U$3.34; no longer U$6.34
- net INH_B: now also U$3.36; no longer U$6.36
- net INH_C: now also U$3.38; no longer U$6.38
- net INL_A: now also U$3.35; no longer U$6.35
- net INL_B: now also U$3.37; no longer U$6.37
- net INL_C: now also U$3.39; no longer U$6.39
- net N$12: now also C12.2, U$3.7; no longer C8.2, U$6.7
- net N$13: now also C7.1, U$3.2; no longer C3.1, U$6.2
- net N$2: now also R10.2, R6.1, U$3.32; no longer R5.1, R9.2, U$6.32
- net N$21: now also C5.1, U$3.42; no longer U$6.42
- net N$22: now also C8.2, U$3.4; no longer C6.2, U$6.4
- net N$23: now also C8.1, U$3.3; no longer C6.1, U$6.3
- net N$4: now also R3.1, U$3.48; no longer R4.1, U$3.1
- net N$5: now also R11.2, R7.1, U$3.31; no longer R10.2, R6.1, U$6.31
- net N$6: now also C5.2, U$3.45; no longer R2.1
- net N$7: now also R12.2, R8.1, U$3.30; no longer R11.2, R7.1, U$6.30
- net N$8: now also R9.2, U$3.29; no longer R8.2, U$6.29
- net PHASA: now also U$3.9; no longer U$6.9
- net PHASB: now also U$3.16; no longer U$6.16
- net PHASC: now also U$3.19; no longer U$6.19
- net PVDD: now also C10.1, C12.1, C13.1, C16.2, C17.2, C3.2, C6.1, R4.2, U$3.43, U$3.5, U$3.6; no longer C11.1, C13.2, C14.2, C4.1, C7.1, R3.1, U$3.47, U$6.5
- net SN1: now also C14.1, U$3.11; no longer C12.1, U$6.11
- net SN2: now also C18.2, U$3.14; no longer C16.2, U$6.14
- net SO1: now also U$3.23; no longer U$6.23
- net SO2: now also U$3.24; no longer U$6.24
- net VCC: now also R3.2
Routing:
- net PVDD: track 36.5 -> 90.3 mm, vias 66 -> 63
- net CAL: track 39.3 -> 0.00 mm, vias 3 -> 0
- net GND: track 54.6 -> 83.9 mm, vias 70 -> 73
- net PHASC: track 0.00 -> 28.6 mm
- net DVDD: track 31.1 -> 54.3 mm, vias 0 -> 4
- net N$21: track 4.15 -> 26.5 mm, vias 0 -> 2
- net PHASA: track 0.00 -> 22.2 mm
- net INH_A: track 17.8 -> 34.5 mm
- net PHASB: track 0.00 -> 14.9 mm
- net SN1: track 4.15 -> 16.9 mm
- net N$15: track 0.00 -> 8.25 mm
- net N$12: track 0.00 -> 7.42 mm
- net N$4: track 6.02 -> 13.4 mm
- net N$14: track 0.00 -> 6.89 mm
- net N$8: track 0.35 -> 5.78 mm
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Other:
- board text added: "3 Phase Controller - Brad Greer Version 0.3"
- board text removed: "3 Phase Controller - Brad Greer Version 0.2"
